File: KiCad_Files/ShotClockPCB/17pinPCB/17pinPCB.kicad_sch (KiCad schematic)
At the start: 0 parts

Commit message: Initial PCB schematic sans LEDs and buzzer
Parts:
- added C1, C10, C2, C3, C4, C5, C6, C7, C8, C9: 0.1uf, symbol Device:C
- added DS1, DS2, DS3: (no value), ShotClockPCB:TDG1050M, symbol New_Library:TDCG1050M
- added J1: Conn_02x08_Counter_Clockwise, Connector_PinHeader_2.54mm:PinHeader_2x08_P2.54mm_Vertical, symbol Connector_Generic:Conn_02x08_Counter_Clockwise
- added J2: Conn_01x08, Connector_PinHeader_2.54mm:PinHeader_1x08_P2.54mm_Vertical, symbol Connector_Generic:Conn_01x08
- added J3: Conn_02x06_Top_Bottom, symbol Connector_Generic:Conn_02x06_Top_Bottom
- added R1, R2, R3, R4, R5, R6, R7: 10k, symbol Device:R
- added SW1, SW2, SW3, SW4, SW5, SW6, SW7: SW_Push, Button_Switch_THT:SW_PUSH_6mm_H8.5mm, symbol Switch:SW_Push
- added U1: MM74HC154N, Package_DIP:DIP-24_W7.62mm, symbol 74xx:74LS154
- added U3, U4: 74HC04, Package_DIP:DIP-14_W7.62mm, symbol 74xx:74HC04
Connections:
- new net: J1.11 (Pin_11), U1.20 (A3)
- new net: J1.12 (Pin_12), U1.21 (A2)
- new net: J1.13 (Pin_13), U1.22 (A1)
- new net: J1.14 (Pin_14), U1.23 (A0)
- new net: C8.1, U1.24 (VCC)
- new net: C9.2, U4.14 (VCC)
- new net: C10.1, U3.14 (VCC)
- new net +5V: C10.2, C8.2, C9.1, J2.4 (Pin_4), SW1.1, SW2.1, SW3.1, SW4.1, SW5.1, SW6.1, SW7.1
- new net BTN_1: C1.2, J3.1 (Pin_1), R1.1, SW1.2
- new net BTN_2: C2.2, J3.2 (Pin_2), R2.1, SW2.2
- new net BTN_3: C3.2, J3.3 (Pin_3), R3.1, SW3.2
- new net BTN_4: C4.2, J3.4 (Pin_4), R4.1, SW4.2
- new net BTN_5: C5.2, J3.5 (Pin_5), R5.1, SW5.2
- new net BTN_6: C6.2, J3.6 (Pin_6), R6.1, SW6.2
- new net BTN_7: C7.2, J3.7 (Pin_7), R7.1, SW7.2
- new net Colon: DS1.4 (CA_L1_L2), DS2.4 (CA_L1_L2), DS3.4 (CA_L1_L2), J1.9 (Pin_9)
- new net DIG_1: U1.1 (S0), U3.1
- new net DIG_10: U1.10 (S9), U4.9
- new net DIG_10_IN: DS3.2 (CA_D2), U4.8
- new net DIG_11: U1.11 (S10), U4.11
- new net DIG_11_IN: DS3.6 (CA_D3), U4.10
- new net DIG_12: U1.13 (S11), U4.13
- new net DIG_12_IN: DS3.8 (CA_D4), U4.12
- new net DIG_1_IN: DS1.1 (CA_D1), U3.2
- new net DIG_2: U1.2 (S1), U3.3
- new net DIG_2_IN: DS1.2 (CA_D2), U3.4
- new net DIG_3: U1.3 (S2), U3.5
- new net DIG_3_IN: DS1.6 (CA_D3), U3.6
- new net DIG_4: U1.4 (S3), U3.9
- new net DIG_4_IN: DS1.8 (CA_D4), U3.8
- new net DIG_5: U1.5 (S4), U3.11
- new net DIG_5_IN: DS2.1 (CA_D1), U3.10
- new net DIG_6: U1.6 (S5), U3.13
- new net DIG_6_IN: DS2.2 (CA_D2), U3.12
- new net DIG_7: U1.7 (S6), U4.1
- new net DIG_7_IN: DS2.6 (CA_D3), U4.2
- new net DIG_8: U1.8 (S7), U4.3
- new net DIG_8_IN: DS2.8 (CA_D4), U4.4
- new net DIG_9: U1.9 (S8), U4.5
- new net DIG_9_IN: DS3.1 (CA_D1), U4.6
- new net GND: C1.1, C2.1, C3.1, C4.1, C5.1, C6.1, C7.1, DS1.12 (L1_L2), DS1.9 (L3), DS2.12 (L1_L2), DS2.9 (L3), DS3.12 (L1_L2), DS3.9 (L3), J2.3 (Pin_3), R1.2, R2.2, R3.2, R4.2, R5.2, R6.2, R7.2, U1.12 (GND), U1.18 (E0), U1.19 (E1), U3.7 (GND), U4.7 (GND)
- new net SEG_A: DS1.14 (A), DS2.14 (A), DS3.14 (A), J1.1 (Pin_1)
- new net SEG_B: DS1.16 (B), DS2.16 (B), DS3.16 (B), J1.2 (Pin_2)
- new net SEG_C: DS1.13 (C), DS2.13 (C), DS3.13 (C), J1.3 (Pin_3)
- new net SEG_D: DS1.3 (D), DS2.3 (D), DS3.3 (D), J1.4 (Pin_4)
- new net SEG_DP: DS1.7 (DP), DS2.7 (DP), DS3.7 (DP), J1.8 (Pin_8)
- new net SEG_E: DS1.5 (E), DS2.5 (E), DS3.5 (E), J1.5 (Pin_5)
- new net SEG_F: DS1.11 (F), DS2.11 (F), DS3.11 (F), J1.6 (Pin_6)
- new net SEG_G: DS1.15 (G), DS2.15 (G), DS3.15 (G), J1.7 (Pin_7)
- new net Top_Point: DS1.10 (CA_L3), DS2.10 (CA_L3), DS3.10 (CA_L3), J1.10 (Pin_10)
- no-connect marks 0 -> 6

Commit message: Added LED to schematic
Parts:
- removed C7: 0.1uf, symbol Device:C
- removed SW7: SW_Push, Button_Switch_THT:SW_PUSH_6mm_H8.5mm, symbol Switch:SW_Push
- added D1, D2, D3, D4, D5, D6: P2, symbol Device:LED
- added R10, R11, R12, R8, R9: 100R, symbol Device:R
- R7: value 10k -> 100R
Connections:
- net GND: now also D1.1 (K), D2.1 (K), D3.1 (K), D4.1 (K), D5.1 (K), D6.1 (K); no longer R7.2
- net LED_POS_HOME: now reaches J1.15 (Pin_15)
- net LED_POS_HOME: now also R11.2
- net LED_POS_AWAY: now reaches J1.16 (Pin_16)
- net LED_POS_AWAY: now also R12.2
- net LED_P4: now reaches J3.10 (Pin_10)
- net LED_P4: now also R10.2
- net LED_P2: now reaches J3.8 (Pin_8)
- net LED_P2: now also R8.2
- net LED_P3: now reaches J3.9 (Pin_9)
- net LED_P3: now also R9.2
- net BTN_7: no longer names the net of R7.1
- net BTN_7: now also D1.2 (A); no longer J3.7 (Pin_7)
- new net: D6.2 (A), R12.1
- new net: D5.2 (A), R11.1
- new net: D4.2 (A), R10.1
- new net: D2.2 (A), R8.1
- new net: D3.2 (A), R9.1
- new net LED_P1: J3.7 (Pin_7), R7.2

Commit message: finalized PCB design
Parts:
- removed DS1, DS2, DS3: (no value), ShotClockPCB:TDG1050M, symbol New_Library:TDCG1050M
- added BZ1: Buzzer, Buzzer_Beeper:Buzzer_12x9.5RM7.6, symbol Device:Buzzer
- added DS1, DS2, DS3: (no value), ShotClockPCB:TDG1050M, symbol 7_seg_lib:TDCG1050M
- added Q1: Q_NPN_CBE, Package_TO_SOT_THT:TO-92_Inline, symbol Transistor_BJT:Q_NPN_CBE
- added R13: 1k, Resistor_THT:R_Axial_DIN0207_L6.3mm_D2.5mm_P7.62mm_Horizontal, symbol Device:R
- C1, C10, C2, C3, C4, C5, C6, C8, C9: footprint (none) -> Capacitor_THT:C_Disc_D5.0mm_W2.5mm_P5.00mm
- D1: value P2 -> P1; footprint (none) -> LED_THT:LED_D5.0mm
- D2: footprint (none) -> LED_THT:LED_D5.0mm
- D3: value P2 -> P3; footprint (none) -> LED_THT:LED_D5.0mm
- D4: value P2 -> P4; footprint (none) -> LED_THT:LED_D5.0mm
- D5: value P2 -> POS_HOME; footprint (none) -> LED_THT:LED_D5.0mm
- D6: value P2 -> POS_AWAY; footprint (none) -> LED_THT:LED_D5.0mm
- J3: footprint (none) -> Connector_PinHeader_2.54mm:PinHeader_2x06_P2.54mm_Vertical
- R1, R10, R11, R12, R2, R3, R4, R5, R6, R7, R8, R9: footprint (none) -> Resistor_THT:R_Axial_DIN0207_L6.3mm_D2.5mm_P7.62mm_Horizontal
Connections:
- net Top_Point is gone; now on net SEL_A0: J1.10 (Pin_10)
- net +5V: now also C10.1, C9.2, U1.24 (VCC), U3.14 (VCC), U4.14 (VCC), BZ1.1 (+); no longer C10.2, C9.1
- net BTN_1: now also J3.2 (Pin_2); no longer J3.1 (Pin_1)
- net BTN_2: now also J3.4 (Pin_4); no longer J3.2 (Pin_2)
- net BTN_3: now also J3.6 (Pin_6); no longer J3.3 (Pin_3)
- net BTN_4: now also J3.8 (Pin_8); no longer J3.4 (Pin_4)
- net BTN_5: now also J3.10 (Pin_10); no longer J3.5 (Pin_5)
- net BTN_6: now also J3.1 (Pin_1); no longer J3.6 (Pin_6)
- net Colon: now also J1.13 (Pin_13), DS1.4 (CA_L1_L2), DS2.4 (CA_L1_L2), DS3.4 (CA_L1_L2); no longer J1.9 (Pin_9)
- net DIG_10_IN: now also DS3.2 (CA_D2)
- net DIG_11_IN: now also DS3.6 (CA_D3)
- net DIG_12_IN: now also DS3.8 (CA_D4)
- net DIG_1_IN: now also DS1.1 (CA_D1)
- net DIG_2_IN: now also DS1.2 (CA_D2)
- net DIG_3_IN: now also DS1.6 (CA_D3)
- net DIG_4_IN: now also DS1.8 (CA_D4)
- net DIG_5_IN: now also DS2.1 (CA_D1)
- net DIG_6_IN: now also DS2.2 (CA_D2)
- net DIG_7_IN: now also DS2.6 (CA_D3)
- net DIG_8_IN: now also DS2.8 (CA_D4)
- net DIG_9_IN: now also DS3.1 (CA_D1)
- net GND: now also C10.2, C8.1, C9.1, DS1.10 (CA_L3), DS1.12 (L1_L2), DS1.9 (L3), DS2.10 (CA_L3), DS2.12 (L1_L2), DS2.9 (L3), DS3.10 (CA_L3), DS3.12 (L1_L2), DS3.9 (L3), Q1.3 (E)
- net LED_P1: now also J3.3 (Pin_3); no longer J3.7 (Pin_7)
- net LED_P2: now also J3.5 (Pin_5); no longer J3.8 (Pin_8)
- net LED_P3: now also J3.7 (Pin_7); no longer J3.9 (Pin_9)
- net LED_P4: now also J3.9 (Pin_9); no longer J3.10 (Pin_10)
- net LED_POS_AWAY: now also J1.14 (Pin_14); no longer J1.16 (Pin_16)
- net LED_POS_HOME: now also J1.16 (Pin_16); no longer J1.15 (Pin_15)
- net SEG_A: now also J1.2 (Pin_2), DS1.14 (A), DS2.14 (A), DS3.14 (A); no longer J1.1 (Pin_1)
- net SEG_B: now also J1.1 (Pin_1), DS1.16 (B), DS2.16 (B), DS3.16 (B); no longer J1.2 (Pin_2)
- net SEG_C: now also J1.9 (Pin_9), DS1.13 (C), DS2.13 (C), DS3.13 (C); no longer J1.3 (Pin_3)
- net SEG_D: now also J1.3 (Pin_3), DS1.3 (D), DS2.3 (D), DS3.3 (D); no longer J1.4 (Pin_4)
- net SEG_DP: now also J1.7 (Pin_7), DS1.7 (DP), DS2.7 (DP), DS3.7 (DP); no longer J1.8 (Pin_8)
- net SEG_E: now also J1.15 (Pin_15), DS1.5 (E), DS2.5 (E), DS3.5 (E); no longer J1.5 (Pin_5)
- net SEG_F: now also J1.5 (Pin_5), DS1.11 (F), DS2.11 (F), DS3.11 (F); no longer J1.6 (Pin_6)
- net SEG_G: now also J1.11 (Pin_11), DS1.15 (G), DS2.15 (G), DS3.15 (G); no longer J1.7 (Pin_7)
- net SEL_A3: now reaches U1.20 (A3)
- net SEL_A3: now also J1.4 (Pin_4); no longer J1.11 (Pin_11)
- net Buzzer: now reaches J1.12 (Pin_12)
- net Buzzer: now also R13.2; no longer U1.21 (A2)
- net SEL_A1: now reaches U1.22 (A1)
- net SEL_A1: now also J1.8 (Pin_8); no longer J1.13 (Pin_13)
- net SEL_A0: now reaches U1.23 (A0)
- net SEL_A0: no longer J1.14 (Pin_14)
- new net: BZ1.2 (-), Q1.1 (C)
- new net: Q1.2 (B), R13.1
- new net SEL_A2: J1.6 (Pin_6), U1.21 (A2)
- no-connect marks 6 -> 12
Other:
- moved on the sheet: C10, C8, D5, D6, R11, R12
