File: KiCad_Files/ShotClockPCB/17pinPCB/17pinPCB-backups/first_working_design.kicad_pcb (KiCad board)
At the start: 2 copper layers, 94 x 98 mm, 45 parts, among them J1 Conn_02x08_Counter_Clockwise, J2 Conn_01x08, J3 Conn_02x06_Top_Bottom, Q1 Q_NPN_CBE, SW1 SW_Push, SW2 SW_Push, SW3 SW_Push, SW4 SW_Push, SW5 SW_Push, SW6 SW_Push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

Commit message: finalized PCB design
Parts:
- moved R6 2.37 mm to (62.3, 62.1)
- moved SW6 2.37 mm to (57.9, 59.2)
- moved C6 2.37 mm to (57.9, 67.1)
Routing:
- net /BTN_6: track 80.9 -> 82.8 mm
Other:
- board text removed: "+5V"
- board text removed: "4/16/2026 SoCET Intro 1 Team 14"
- board text removed: "AWAY"
- board text removed: "GAME"
- board text removed: "GND"
- board text removed: "HOME"
- board text removed: "SHOT"
Changed lines of the file:
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@@
 		(zone_defaults)
 		(pcbplotparams
-			(layerselection 0x00000000_00000000_55555555_575555ff)
+			(layerselection 0x00000000_00000000_55555555_5755f5ff)
 			(plot_on_all_layers_selection 0x00000000_00000000_00000000_00000000)
 			(disableapertmacros no)
@@
 			(outputformat 1)
 			(mirror no)
-			(drillshape 0)
+			(drillshape 1)
 			(scaleselection 1)
 			(outputdirectory "")
@@
 	(footprint "Button_Switch_THT:SW_PUSH_6mm_H8.5mm"
 		(layer "F.Cu")
-		(at 57.85 61.616899 90)
+		(at 57.85 59.25 90)
 		(descr "tactile push button, 6x6mm e.g. PHAP33xx series, height=8.5mm")
 		(tags "tact sw push 6mm")
@@
 	(footprint "Capacitor_THT:C_Disc_D5.0mm_W2.5mm_P5.00mm"
 		(layer "F.Cu")
-		(at 57.8926 69.459499 90)
+		(at 57.8926 67.0926 90)
 		(descr "C, Disc series, Radial, pin pitch=5.00mm, diameter*width=5*2.5mm^2, Capacitor, http://cdn-reichelt.de/documents/datenblatt/B300/DS_KERKO_TC.pdf")
 		(tags "C Disc series Radial pin pitch 5.00mm diameter 5mm width 2.5mm Capacitor")
 		(property "Reference" "C6"
-			(at 4.459499 -2.6926 90)
+			(at 2.5 -2.5 90)
 			(layer "F.SilkS")
 			(effects
@@
 	(footprint "Resistor_THT:R_Axial_DIN0207_L6.3mm_D2.5mm_P7.62mm_Horizontal"
 		(layer "F.Cu")
-		(at 62.3046 64.461699 -90)
+		(at 62.3046 62.0948 -90)
 		(descr "Resistor, Axial_DIN0207 series, Axial, Horizontal, pin pitch=7.62mm, 0.25W = 1/4W, length*diameter=6.3*2.5mm^2, http://cdn-reichelt.de/documents/datenblatt/B400/1_4W%23YAG.pdf")
 		(tags "Resistor Axial_DIN0207 series Axial Horizontal pin pitch 7.62mm 0.25W = 1/4W length 6.3mm diameter 2.5mm")
@@
 		(layer "Edge.Cuts")
 	)
-	(gr_text "+5V"
-		(at 40 107.9 0)
-		(layer "F.Cu")
-		(effects
-			(font
-				(size 1.5 1.5)
-				(thickness 0.3)
-				(bold yes)
-			)
-			(justify left bottom)
-		)
-	)
-	(gr_text "GND"
-		(at 53.7 114.2 0)
-		(layer "F.Cu")
-		(effects
-			(font
-				(size 1.5 1.5)
-				(thickness 0.3)
-				(bold yes)
-			)
-			(justify left bottom)
-		)
-	)
-	(gr_text "4/16/2026    SoCET Intro 1    Team 14"
-		(at 37.1 148.1 0)
-		(layer "F.SilkS")
-		(effects
-			(font
-				(size 1 1)
-				(thickness 0.1)
-			)
-			(justify left bottom)
-		)
-	)
-	(gr_text "SHOT"
-		(at 87.4 57.4641 270)
-		(layer "F.SilkS")
-		(effects
-			(font
-				(size 1 1)
-				(thickness 0.1)
-			)
-			(justify left bottom)
-		)
-	)
-	(gr_text "AWAY"
-		(at 104.1 88.8 270)
-		(layer "F.SilkS")
-		(effects
-			(font
-				(size 1 1)
-				(thickness 0.1)
-			)
-			(justify left bottom)
-		)
-	)
-	(gr_text "HOME"
-		(at 104.2 57.2 270)
-		(layer "F.SilkS")
-		(effects
-			(font
-				(size 1 1)
-				(thickness 0.1)
-			)
-			(justify left bottom)
-		)
-	)
-	(gr_text "GAME"
-		(at 121.3 57.1 270)
-		(layer "F.SilkS")
-		(effects
-			(font
-				(size 1 1)
-				(thickness 0.1)
-			)
-			(justify left bottom)
-		)
-	)
 	(segment
 		(start 46.7 67.59)
@@
 	)
 	(segment
-		(start 59.6824 69.459499)
-		(end 62.3046 72.081699)
-		(width 0.5)
-		(layer "F.Cu")
-		(net "GND")
-	)
-	(segment
 		(start 59.0114 106.1781)
 		(end 58.225 105.3917)
@@
 	)
 	(segment
+		(start 62.3046 69.7148)
+		(end 59.6824 67.0926)
+		(width 0.5)
+		(layer "F.Cu")
+		(net "GND")
+	)
+	(segment
 		(start 58.225 96.57)
 		(end 58.225 105.3917)
@@
 	)
 	(segment
+		(start 57.8926 67.0926)
+		(end 57.9926 67.0926)
+		(width 0.5)
+		(layer "F.Cu")
+		(net "GND")
+	)
+	(segment
 		(start 54.205 67.705)
 		(end 54.11 67.61)
@@
 	)
 	(segment
-		(start 57.8926 69.459499)
-		(end 59.6824 69.459499)
-		(width 0.5)
-		(layer "F.Cu")
-		(net "GND")
-	)
-	(segment
 		(start 54.31 76.458)
 		(end 54.21 76.358)
@@
 	)
 	(segment
+		(start 59.6824 67.0926)
+		(end 57.9926 67.0926)
+		(width 0.5)
+		(layer "F.Cu")
+		(net "GND")
+	)
+	(segment
 		(start 57.5 133.8733)
 		(end 59.0114 132.3619)
@@
 	)
 	(segment
-		(start 54.21 67.7)
-		(end 56.133101 67.7)
-		(width 0.5)
-		(layer "B.Cu")
-		(net "GND")
-	)
-	(segment
 		(start 121.6778 75.8956)
 		(end 121.6778 76.9382)
@@
 	)
 	(segment
+		(start 54.8174 67.0926)
+		(end 54.21 67.7)
+		(width 0.5)
+		(layer "B.Cu")
+		(net "GND")
+	)
+	(segment
 		(start 51.7 80.3)
 		(end 55.5433 80.3)
@@
 	)
 	(segment
-		(start 56.133101 67.7)
-		(end 57.8926 69.459499)
-		(width 0.5)
-		(layer "B.Cu")
-		(net "GND")
-	)
-	(segment
 		(start 105.6878 82.7121)
 		(end 104.4757 81.5)
@@
 	)
 	(segment
+		(start 57.8926 67.0926)
+		(end 54.8174 67.0926)
+		(width 0.5)
+		(layer "B.Cu")
+		(net "GND")
+	)
+	(segment
 		(start 86.9558 80.2854)
 		(end 63.1674 80.2854)
@@
 	)
 	(segment
+		(start 57.85 52.75)
+		(end 54.65 52.75)
+		(width 0.5)
+		(layer "F.Cu")
+		(net "+5V")
+	)
+	(segment
 		(start 112.485 127.96)
 		(end 112.605 128.08)
@@
 	)
 	(segment
-		(start 120.4132 143.3285)
-		(end 121.8781 144.7934)
+		(start 54.65 52.75)
+		(end 53.7071 53.6929)
 		(width 0.5)
 		(layer "F.Cu")
@@
 	)
 	(segment
-		(start 49.6013 121.247)
-		(end 48.8 122.0483)
+		(start 57.85 57.8358)
+		(end 57.85 59.25)
 		(width 0.5)
 		(layer "F.Cu")
@@
 	)
 	(segment
-		(start 94.385 127.96)
-		(end 92.735 126.31)
+		(start 120.4132 143.3285)
+		(end 121.8781 144.7934)
 		(width 0.5)
 		(layer "F.Cu")
@@
 	)
 	(segment
-		(start 44.75 53.45)
-		(end 56.183101 53.45)
+		(start 49.6013 121.247)
+		(end 48.8 122.0483)
 		(width 0.5)
 		(layer "F.Cu")
@@
 	)
 	(segment
-		(start 43.55 54.65)
-		(end 44.75 53.45)
+		(start 94.385 127.96)
+		(end 92.735 126.31)
 		(width 0.5)
 		(layer "F.Cu")
@@
 	)
 	(segment
-		(start 57.8926 62.0926)
-		(end 58.5148 62.0926)
-		(width 0.3)
-		(layer "F.Cu")
-		(net "+5V")
-	)
-	(segment
 		(start 94.465 131.34)
 		(end 94.385 131.26)
@@
 	)
 	(segment
-		(start 112.605 128.08)
-		(end 112.605 131.34)
+		(start 53.7071 53.6929)
+		(end 57.85 57.8358)
 		(width 0.5)
 		(layer "F.Cu")
@@
 	)
 	(segment
-		(start 56.183101 53.45)
-		(end 57.85 55.116899)
+		(start 112.605 128.08)
+		(end 112.605 131.34)
 		(width 0.5)
 		(layer "F.Cu")
@@
 	)
 	(segment
-		(start 57.85 61.616899)
-		(end 57.85 55.116899)
+		(start 53.4642 53.45)
+		(end 53.7071 53.6929)
+		(width 0.5)
+		(layer "F.Cu")
+		(net "+5V")
+	)
+	(segment
+		(start 44.75 53.45)
+		(end 53.4642 53.45)
+		(width 0.5)
+		(layer "F.Cu")
+		(net "+5V")
+	)
+	(segment
+		(start 43.55 54.65)
+		(end 44.75 53.45)
 		(width 0.5)
 		(layer "F.Cu")
@@
 	)
 	(segment
-		(start 57.8926 64.459499)
-		(end 56.695601 64.459499)
+		(start 62.35 59.25)
+		(end 62.35 62.0494)
 		(width 0.3)
 		(layer "F.Cu")
@@
 	)
 	(segment
-		(start 62.35 55.116899)
-		(end 62.35 61.616899)
+		(start 58.5148 62.0926)
+		(end 62.3023 62.0926)
 		(width 0.3)
 		(layer "F.Cu")
@@
 	)
 	(segment
-		(start 62.35 61.616899)
-		(end 62.35 64.416299)
+		(start 57.8926 62.0926)
+		(end 58.5148 62.0926)
 		(width 0.3)
 		(layer "F.Cu")
@@
 	)
 	(segment
-		(start 62.35 62.0494)
-		(end 62.3046 62.0948)
+		(start 56.3551 64.2523)
+		(end 56.3551 105.2583)
 		(width 0.3)
 		(layer "F.Cu")
@@
 	)
 	(segment
-		(start 62.3023 62.0926)
-		(end 62.3046 62.0948)
+		(start 62.35 52.75)
+		(end 62.35 59.25)
 		(width 0.3)
 		(layer "F.Cu")
@@
 	)
 	(segment
-		(start 56.695601 64.459499)
-		(end 56.3551 64.8)
+		(start 62.35 62.0494)
+		(end 62.3046 62.0948)
 		(width 0.3)
 		(layer "F.Cu")
@@
 	)
 	(segment
-		(start 39.84 123.38)
-		(end 39.84 122.1783)
+		(start 62.3023 62.0926)
+		(end 62.3046 62.0948)
 		(width 0.3)
 		(layer "F.Cu")
@@
 	)
 	(segment
-		(start 62.3024 64.459499)
-		(end 62.3046 64.461699)
+		(start 39.84 123.38)
+		(end 39.84 122.1783)
 		(width 0.3)
 		(layer "F.Cu")
@@
 	)
 	(segment
-		(start 57.8926 64.459499)
-		(end 62.3024 64.459499)
-		(width 0.3)
-		(layer "F.Cu")
-		(net "/BTN_6")
-	)
-	(segment
-		(start 56.3551 64.8)
-		(end 56.3551 105.2583)
+		(start 58.5148 62.0926)
+		(end 56.3551 64.2523)
 		(width 0.3)
 		(layer "F.Cu")
@@
 		(width 0.3)
 		(layer "F.Cu")
-		(net "/BTN_6")
-	)
-	(segment
-		(start 62.35 64.416299)
-		(end 62.3046 64.461699)
-		(width 0.3)
-		(layer "F.Cu")
